Commit message: Before new driver installation

File: tara_firmware/tf/tara.urdf (robot description, URDF)
Before this commit: robot tara_mobile, 6 links, 5 joints
Links:
- link base_link: geometry visual box size=0.5588 0.5588 0.33
- link lwheel: geometry visual cylinder length=0.050 radius=0.1551
- link rwheel: geometry visual cylinder length=0.050 radius=0.1551
Joints:
- joint base_to_lwheel: origin xyz=0 0.115 0.046 rpy=1.5708 0 0 -> xyz=0 0.42164 0.1651 rpy=1.5708 0 0
- joint base_to_rwheel: origin xyz=0 -0.115 0.046 rpy=-1.5708 0 0 -> xyz=0 -0.42164 0.1651 rpy=-1.5708 0 0

Commit message: Bug fixes

File: tara_firmware/tf/tara.urdf (robot description, URDF)
Before this commit: robot tara_mobile, 1 links, 0 joints
Links:
- added link fwheel; visual cylinder length=0.005 radius=0.020
- added link fwheel_attach; visual cylinder length=0.060 radius=0.023
- added link lwheel; visual cylinder length=0.008 radius=0.046
- added link rwheel; visual cylinder length=0.008 radius=0.046
- added link scanner; visual box size=0.015 0.045 0.015
- link base_link: geometry visual box size=0.16 0.16 0.12
Joints:
- added joint base_to_fattach: type fixed, parent base_link, child fwheel_attach, origin xyz=0 0 0 rpy=0 0 0
- added joint base_to_fwheel: type fixed, parent base_link, child fwheel, origin xyz=0.13 0 0.02 rpy=0 0 0
- added joint base_to_lwheel: type fixed, parent base_link, child lwheel, origin xyz=0 0.115 0.046 rpy=1.5708 0 0
- added joint base_to_rwheel: type fixed, parent base_link, child rwheel, origin xyz=0 -0.115 0.046 rpy=-1.5708 0 0
- added joint base_to_scanner: type fixed, parent base_link, child scanner, origin xyz=0.105 0 0.22 rpy=0 0 0
